File: PCB/V1/V1.kicad_sch (KiCad schematic)
At the start: 1 part, among them U1 MDBT50Q-1MV2

Commit message: udated by FZ
Parts:
- removed U1: MDBT50Q-1MV2, RF_Module:Raytac_MDBT50Q, symbol RF_Module:MDBT50Q-1MV2
- added C1, C3: 10uF, Capacitor_SMD:C_1206_3216Metric_Pad1.33x1.80mm_HandSolder, symbol Device:C_Small
- added C2, C4: 22pF, Capacitor_SMD:C_0402_1005Metric_Pad0.74x0.62mm_HandSolder, symbol Device:C_Small
- added C5, C6: 10uF, Capacitor_SMD:C_0402_1005Metric_Pad0.74x0.62mm_HandSolder, symbol Device:C_Small
- added C7: 0.1uF, Capacitor_SMD:C_0402_1005Metric_Pad0.74x0.62mm_HandSolder, symbol Device:C_Small
- added D1: RED, LED_SMD:LED_0603_1608Metric_Pad1.05x0.95mm_HandSolder, symbol Device:LED_Small_Filled
- added D2: LED, Diode_SMD:D_0603_1608Metric_Pad1.05x0.95mm_HandSolder, symbol Device:LED
- added F1: Fuse_Small, Fuse:Fuse_1206_3216Metric_Pad1.42x1.75mm_HandSolder, symbol Device:Fuse_Small
- added J2: USB3131-30-0230-A_REVB, Mylib:GCT_USB3131-30-0230-A_REVB, symbol USB3131-30-0230-A_REVB:USB3131-30-0230-A_REVB
- added J4: Programmer, Connector_PinHeader_2.54mm:PinHeader_1x02_P2.54mm_Vertical, symbol Connector:Conn_01x02_Male
- added J5, J6: Conn_02x06_Odd_Even, Connector_PinHeader_2.54mm:PinHeader_2x06_P2.54mm_Vertical, symbol Connector_Generic:Conn_02x06_Odd_Even
- added J7, J8: RESET, Connector_PinHeader_2.00mm:PinHeader_1x02_P2.00mm_Vertical, symbol Connector:Conn_01x02_Pin
- added L1: 10uH, Inductor_SMD:L_0603_1608Metric_Pad1.05x0.95mm_HandSolder, symbol Device:L_Small
- added R1, R2: 4.7K, Resistor_SMD:R_0402_1005Metric_Pad0.72x0.64mm_HandSolder, symbol Device:R_Small
- added R10: 1M, Resistor_SMD:R_0603_1608Metric_Pad0.98x0.95mm_HandSolder, symbol Device:R_Small
- added R11, R14: 330, Resistor_SMD:R_0402_1005Metric_Pad0.72x0.64mm_HandSolder, symbol Device:R_Small
- added R4: 10K, Resistor_SMD:R_0402_1005Metric, symbol Device:R_Small
- added R7, R8: 499K, Resistor_SMD:R_0402_1005Metric_Pad0.72x0.64mm_HandSolder, symbol Device:R_Small
- added S1: TL1105F160Q, Mylib:SW_TL1105F160Q, symbol TL1105F160Q:TL1105F160Q
- added S2, S3: SS12D07VG4, Mylib:SW_SS12D07VG4, symbol SS12D07VG4:SS12D07VG4
- added TP4, TP5, TP6: TestPoint, TestPoint:TestPoint_Pad_1.5x1.5mm, symbol Connector:TestPoint
- added U2: MDBT50Q-1MV2, Mylib:XCVR_MDBT50Q-1MV2, symbol MDBT50Q-1MV2:MDBT50Q-1MV2
- added Y1: 32.768kHz, Capacitor_SMD:C_0805_2012Metric_Pad1.18x1.45mm_HandSolder, symbol Device:Crystal_Small
Connections:
- new net: D2.1 (K), TP5.1
- new net: D2.2 (A), TP6.1
- new net: D1.1 (K), R11.1
- new net: C2.2, U2.17 (P0.00/XL1), Y1.2
- new net: C4.2, U2.18 (P0.01/XL2), Y1.1
- new net: L1.2, U2.31 (DCCH)
- new net: J7.1 (Pin_1), S2.2
- new net: J7.2 (Pin_2), S2.3
- new net: J8.1 (Pin_1), S1.1
- new net: J8.2 (Pin_2), S1.3
- new net: F1.2, J2.1 (VCC)
- new net +5V: C1.1, C3.1, F1.1, J5.5 (Pin_5), R10.2, U2.32 (VBUS)
- new net A0: U2.20 (P0.04/AIN2)
- new net A1: U2.21 (P0.05/AIN3)
- new net A2: J5.6 (Pin_6), R7.2, R8.1, U2.14 (P0.30/AIN6)
- new net A3: J5.4 (Pin_4), U2.13 (P0.28/AIN4), U2.46 (P0.22)
- new net A4: J6.8 (Pin_8), U2.11 (P0.02/AIN0)
- new net A5: J5.3 (Pin_3), U2.9 (P0.03/AIN1)
- new net D1: J6.4 (Pin_4)
- new net D10: C7.1, J6.2 (Pin_2), R14.1, U2.16 (P0.27)
- new net D11: U2.22 (P0.06)
- new net D12: J6.1 (Pin_1), U2.24 (P0.08)
- new net D13: U2.26 (P1.09/TRACEDATA3)
- new net D2: J6.7 (Pin_7), R4.1, U2.54 (P0.10/NFC2)
- new net D3: J6.6 (Pin_6)
- new net D4: J6.11 (Pin_11)
- new net D5: U2.25 (P1.08)
- new net D6: U2.23 (P0.07/TRACECLK)
- new net D8: J5.2 (Pin_2)
- new net D9: U2.19 (P0.26)
- new net GND: C1.2, C2.1, C3.2, C4.1, C5.1, C6.1, C7.2, J2.5 (GND), J2.S1 (SHIELD), J2.S2 (SHIELD), J5.10 (Pin_10), J5.8 (Pin_8), J6.10 (Pin_10), J6.12 (Pin_12), R10.1, R11.2, R4.2, R8.2, S2.S1 (SHIELD), S2.S2 (SHIELD), S3.3, S3.S1 (SHIELD), S3.S2 (SHIELD), U2.1 (GND), U2.15 (GND), U2.2 (GND), U2.33 (GND), U2.55 (GND)
- new net LED1: D1.2 (A), U2.8 (P1.15)
- new net LED2: U2.3 (P1.10)
- new net LORA_FREQ_SELECT: R14.2, S3.2
- new net MISO: J6.9 (Pin_9), U2.39 (P0.15)
- new net MOSI: J6.3 (Pin_3), U2.37 (P0.13)
- new net RXD: J5.7 (Pin_7), U2.48 (P0.24)
- new net SCK: J6.5 (Pin_5), U2.36 (P0.14)
- new net SCL: J5.12 (Pin_12), R2.1, U2.27 (P0.11/TRACEDATA2)
- new net SDA: J5.11 (Pin_11), R1.1, U2.29 (P0.12/TRACEDATA1)
- new net SWDCLK: J4.1 (Pin_1), U2.53 (SWDCLK)
- new net SWDIO: J4.2 (Pin_2), U2.51 (SWDIO)
- new net TXD: J5.9 (Pin_9), U2.49 (P0.25)
- new net USB+: J2.3 (D+), U2.35 (D+)
- new net USB-: J2.2 (D-), U2.34 (D-)
- new net VBAT: J5.1 (Pin_1), R7.1, TP4.1
- new net VCC: C5.2, C6.2, L1.1, R1.2, R2.2, U2.28 (VDD), U2.30 (VDDH)
- new net ~{CS}: U2.38 (P0.16)
- new net ~{RESET}: U2.40 (P0.18/~{RESET})
- no-connect marks 0 -> 25
Other:
- note added: "Connector"
- note added: "IMU"
- note added: "LoRa frequency switch"
- note added: "Microcontroller"
- note added: "Power switch"
- note added: "Reset switch"
- note added: "SSQ-106-23-G-D"
- note added: "USB"
- company: (none) -> MIT Media Lab
- title: (none) -> HexSense Svalbard - MCU module
