File: PCB/MCU/V1/V1.kicad_pcb (KiCad board)
At the start: 2 copper layers, 29 x 23 mm, 36 parts, among them J1 encoder, J2 buttons, J3 joystick, Q1 PJE8408_R1_00001, Q2 PJE8408_R1_00001, U1 BC832, U2 ICM-20948, U3 AP2112K-3.3, U4 AP2112K-1.8, Y1 32.768kHz

Commit message: udated by FZ
Parts:
- moved J3 2.01 mm to (162.3, 101.3)
- moved R10 2.01 mm to (167.3, 103.7)
- moved R12 2.01 mm to (165.3, 103.7)
- moved R13 2.01 mm to (163.3, 103.7)
- moved R14 2.01 mm to (161.3, 103.7)
- moved R15 2.01 mm to (159.3, 103.7)
- moved R16 2.01 mm to (157.3, 103.7)
Routing:
- net /A2: track 15.9 -> 18.0 mm
- net /A0: track 12.1 -> 14.2 mm
- net /A4: track 22.4 -> 24.5 mm
- net /A1: track 16.1 -> 18.1 mm
- net /A5: track 23.7 -> 25.8 mm
- net /A3: track 19.9 -> 21.9 mm
- net VCC: track 63.9 -> 62.5 mm
- net GND: vias 47 -> 43
