File: PCB/MCU/V1/V1.kicad_pcb (KiCad board)
At the start: 2 copper layers, 30 parts, among them J4 Programmer, J5 Conn_02x06_Odd_Even, J6 Conn_02x06_Odd_Even, J8 RESET, U1 BC832, U2 ICM-20948, Y1 32.768kHz

Commit message: udated by FZ
Parts:
- removed D2: LED, Diode_SMD:D_0603_1608Metric_Pad1.05x0.95mm_HandSolder
- removed J4: Programmer, Connector_PinHeader_2.54mm:PinHeader_1x02_P2.54mm_Vertical
- removed J5, J6: Conn_02x06_Odd_Even, Connector_PinHeader_2.54mm:PinHeader_2x06_P2.54mm_Vertical
- removed J8: RESET, Connector_PinHeader_2.00mm:PinHeader_1x02_P2.00mm_Vertical
- removed L1: 10uH, Inductor_SMD:L_0603_1608Metric_Pad1.05x0.95mm_HandSolder
- removed R4: 10K, Resistor_SMD:R_0402_1005Metric
- removed TP4, TP5, TP6: TestPoint, TestPoint:TestPoint_Pad_1.5x1.5mm
- added C8: 0.1uF, Capacitor_SMD:C_0402_1005Metric_Pad0.74x0.62mm_HandSolder, F.Cu at (198.3, 107.8)
- added J1: encoder, SamacSys_Parts:BM03BSRSSTBTLFSN, F.Cu at (173.8, 112.0)
- added J2: buttons, SamacSys_Parts:BM10BSRSSTBLFSN, F.Cu at (187.0, 113.0)
- added Q1: PJE8408_R1_00001, SamacSys_Parts:SOTFL50P160X60-3N, F.Cu at (184.9, 103.1)
- added Q2: PJE8408_R1_00001, SamacSys_Parts:SOTFL50P160X60-3N, F.Cu at (184.9, 100.9)
- added U3: AP2112K-3.3, Package_TO_SOT_SMD:SOT-23-5, F.Cu at (180.9, 106.0)
- added U4: AP2112K-1.8, Package_TO_SOT_SMD:SOT-23-5, F.Cu at (172.9, 104.2)
- D1: moved to B.Cu
- moved R2 40.9 mm to (187.3, 103.1)
- moved R1 40.9 mm to (187.3, 100.9)
- moved U1 39.3 mm to (194.3, 102.0), turned to -90 degrees
- moved R11 38.8 mm to (187.0, 99.3)
- moved R5 37.7 mm to (184.7, 104.7)
- moved R8 37.4 mm to (185.3, 106.5), turned to 90 degrees
- moved R6 36.4 mm to (184.7, 99.3)
- moved R7 34.9 mm to (181.9, 108.3)
- moved R3 30.3 mm to (176.5, 103.7)
- moved C2 25.9 mm to (186.4, 106.5), turned to -90 degrees
- moved R14 24.9 mm to (172.6, 99.0)
- moved C4 24.2 mm to (185.8, 108.3)
- moved C5 20.7 mm to (184.1, 106.5), turned to -90 degrees
- moved D1 17.3 mm to (187.2, 98.0)
- moved C1 17.3 mm to (176.5, 102.2), turned to 180 degrees
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Connections:
- C5 pad 1: GND -> VCC
- C5 pad 2: VCC -> GND
- C6 pad 1: GND -> +1V8
- C6 pad 2: VCC -> GND
- R14 pad 2: /LORA_FREQ_SELECT -> unconnected-(R14-Pad2)
- R7 pad 2: /A2 -> /BAT_V
- R8 pad 1: /A2 -> /BAT_V
- U1 pad 1: unconnected-(U1-GND-Pad1) -> GND
- U1 pad 13: unconnected-(U1-P02/AIN0-Pad13) -> /BAT_V
- U1 pad 14: unconnected-(U1-P27/SCL-Pad14) -> /SCL
- U1 pad 15: unconnected-(U1-P26/SDA-Pad15) -> /SDA
- U1 pad 16: unconnected-(U1-VDD-Pad16) -> VCC
- U1 pad A5: unconnected-(U1-P08-PadA5) -> /LED1
Routing:
- net VCC: track 0.00 -> 36.0 mm, vias 0 -> 3
- net +1V8: track 0.00 -> 32.6 mm, vias 0 -> 4
- net /VBAT: track 0.00 -> 26.2 mm, vias 0 -> 2
- net /BAT_V: track 0.00 -> 15.1 mm, vias 0 -> 2
- net /SDA: track 0.00 -> 15.0 mm
- net /BTN_1: track 0.00 -> 14.8 mm, vias 0 -> 1
- net /BTN_2: track 0.00 -> 14.1 mm, vias 0 -> 1
- net /SCL: track 0.00 -> 12.0 mm
- net Net-(U2-~{CS}): track 0.00 -> 12.0 mm, vias 0 -> 2
- net Net-(U1-P01/XL2): track 0.00 -> 8.92 mm
- net Net-(U1-P00/XL1): track 0.00 -> 8.32 mm
- net /BTN_3: track 0.00 -> 7.14 mm, vias 0 -> 1
- net /SDA_1V8: track 0.00 -> 6.58 mm
- net /SCL_1V8: track 0.00 -> 5.40 mm
- net /SWDIO: track 0.00 -> 3.98 mm, vias 0 -> 1
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- added copper zone on B.Cu, net GND
- added copper zone on F.Cu, net GND
Other:
- board outline added: 29 x 23 mm
- board text removed: "X"
- board text removed: "Y"
- board text removed: "Z"

Commit message: udated by FZ
Parts:
- added C10: 0.1uF, Capacitor_SMD:C_0402_1005Metric_Pad0.74x0.62mm_HandSolder, F.Cu at (175.4, 108.8)
- added C9: 0.1uF, Capacitor_SMD:C_0402_1005Metric_Pad0.74x0.62mm_HandSolder, F.Cu at (173.1, 108.8)
- added R4: 10K, Resistor_SMD:R_0402_1005Metric_Pad0.72x0.64mm_HandSolder, F.Cu at (173.1, 107.7)
- added R9: 10K, Resistor_SMD:R_0402_1005Metric_Pad0.72x0.64mm_HandSolder, F.Cu at (175.4, 107.7)
- moved U3 0.35 mm to (180.9, 106.4)
- moved R7 0.35 mm to (181.9, 108.6)
Connections:
- J1 pad 1: unconnected-(J1-Pad1) -> GND
- J1 pad 2: unconnected-(J1-Pad2) -> /EN_A
- J1 pad 3: unconnected-(J1-Pad3) -> /EN_B
- J2 pad 10: unconnected-(J2-Pad10) -> GND
- J2 pad 3: /BTN_1 -> /SWDIO
- J2 pad 4: /BTN_2 -> /SWDCLK
- J2 pad 5: /BTN_3 -> /BTN_1
- J2 pad 6: /BTN_4 -> /BTN_2
- J2 pad 7: unconnected-(J2-Pad7) -> /BTN_3
- J2 pad 8: unconnected-(J2-Pad8) -> /BTN_4
- U1 pad B5: unconnected-(U1-P07-PadB5) -> /BTN_1
- U1 pad C5: unconnected-(U1-P09-PadC5) -> /BTN_2
- U1 pad D4: unconnected-(U1-P14-PadD4) -> /BTN_4
- U1 pad D5: unconnected-(U1-P10-PadD5) -> /BTN_3
Routing:
- net /SWDCLK: track 1.52 -> 33.9 mm, vias 1 -> 2
- net /SWDIO: track 3.98 -> 34.8 mm, vias 1 -> 2
- net VCC: track 36.0 -> 50.1 mm
- net /BTN_4: track 1.55 -> 9.83 mm, vias 1 -> 2
- net /EN_B: track 0.00 -> 5.80 mm, vias 0 -> 1
- net /EN_A: track 0.00 -> 5.60 mm, vias 0 -> 1
- net /BTN_3: track 7.14 -> 11.0 mm, vias 1 -> 2
- net unconnected-(U1-P21/RESET-Pad10): track 3.04 -> 0.00 mm, vias 1 -> 0
- net unconnected-(U1-P03/AIN1-Pad9): track 2.47 -> 0.00 mm, vias 1 -> 0
- net /BTN_2: track 14.1 -> 13.2 mm, vias 1 -> 2
- net unconnected-(U1-P07-PadB5): track 0.82 -> 0.00 mm, vias 1 -> 0
- net unconnected-(U1-P09-PadC5): track 0.80 -> 0.00 mm, vias 1 -> 0
- net unconnected-(U1-P10-PadD5): track 0.80 -> 0.00 mm, vias 1 -> 0
- net unconnected-(U1-P14-PadD4): track 0.77 -> 0.00 mm, vias 1 -> 0
- net /BTN_1: track 14.8 -> 15.2 mm, vias 1 -> 2
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
Commit message: udated by FZ
Connections:
- U1 pad D3: unconnected-(U1-P16-PadD3) -> /VIB_CTRL
Routing:
- net unconnected-(U1-P16-PadD3): track 0.84 -> 0.00 mm, vias 1 -> 0
- net /VIB_CTRL: track 0.00 -> 0.84 mm, vias 0 -> 1
- net unconnected-(J2-Pad9): vias 1 -> 0
- net GND: vias 13 -> 9
