File: PCB/MCU/V1/V1.kicad_sch (KiCad schematic)
At the start: 33 parts, among them J4 Programmer, J5 Conn_02x06_Odd_Even, J6 Conn_02x06_Odd_Even, J8 RESET, Q1 PJE8408_R1_00001, Q2 PJE8408_R1_00001, U1 BC832, U2 ICM-20948, Y1 32.768kHz

Commit message: udated by FZ
Parts:
- removed D2: LED, Diode_SMD:D_0603_1608Metric_Pad1.05x0.95mm_HandSolder, symbol Device:LED
- removed J4: Programmer, Connector_PinHeader_2.54mm:PinHeader_1x02_P2.54mm_Vertical, symbol Connector:Conn_01x02_Male
- removed J5, J6: Conn_02x06_Odd_Even, Connector_PinHeader_2.54mm:PinHeader_2x06_P2.54mm_Vertical, symbol Connector_Generic:Conn_02x06_Odd_Even
- removed J8: RESET, Connector_PinHeader_2.00mm:PinHeader_1x02_P2.00mm_Vertical, symbol Connector:Conn_01x02_Pin
- removed L1: 10uH, Inductor_SMD:L_0603_1608Metric_Pad1.05x0.95mm_HandSolder, symbol Device:L_Small
- removed S1: TL1105F160Q, Mylib:SW_TL1105F160Q, symbol TL1105F160Q:TL1105F160Q
- removed TP4, TP5, TP6: TestPoint, TestPoint:TestPoint_Pad_1.5x1.5mm, symbol Connector:TestPoint
- added J1: encoder, SamacSys_Parts:BM03BSRSSTBTLFSN, symbol SamacSys_Parts:BM03B-SRSS-TBT_LF__SN_
- added J2: buttons, BM10BSRSSTBLFSN, symbol SamacSys_Parts:BM10B-SRSS-TB__LF__SN_
- added U3: AP2112K-3.3, Package_TO_SOT_SMD:SOT-23-5, symbol Regulator_Linear:AP2112K-3.3
- added U4: AP2112K-1.8, Package_TO_SOT_SMD:SOT-23-5, symbol Regulator_Linear:AP2112K-1.8
- U1: footprint XCVR_BC832 -> Mylib:XCVR_BC832
Connections:
- net +3.3V is gone; now on net VCC: C8.1, U1.16 (VDD)
- net +1V8: now also C6.1, U4.5 (VOUT)
- net GND: now also C5.2, C6.2, J1.MP1, J1.MP2, J2.MP1, J2.MP2, U3.2 (GND), U4.2 (GND); no longer C5.1, C6.1
- net LED1: now also U1.A5 (P08)
- net VBAT: now also J2.1, U3.1 (VIN), U3.3 (EN), U4.1 (VIN), U4.3 (EN)
- net VCC: now also C5.1, J2.2, U3.5 (VOUT); no longer C5.2, C6.2
- net LORA_FREQ_SELECT: no longer names the net of R14.2
- new net BTN_1: J2.3
- new net BTN_2: J2.4
- new net BTN_3: J2.5
- new net BTN_4: J2.6
- no-connect marks 9 -> 7
Other:
- note removed: "Reset switch"
- note removed: "SSQ-106-23-G-D"
- moved on the sheet: C1, C2, C3, C4, C8, D1, Q1, Q2, R1, R11, R2, R3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

Commit message: udated by FZ
Parts:
- added C10, C9: 0.1uF, Capacitor_SMD:C_0402_1005Metric_Pad0.74x0.62mm_HandSolder, symbol Device:C_Small
- added R4, R9: 10K, Resistor_SMD:R_0402_1005Metric_Pad0.72x0.64mm_HandSolder, symbol Device:R_Small
Connections:
- net BTN_1: now also J2.5, U1.B5 (P07); no longer J2.3
- net BTN_2: now also J2.6, U1.C5 (P09); no longer J2.4
- net BTN_3: now also J2.7, U1.D5 (P10); no longer J2.5
- net BTN_4: now also J2.8, U1.D4 (P14); no longer J2.6
- net GND: now also J1.1, J2.10, C10.1, C9.1
- net SWDCLK: now also J2.4
- net SWDIO: now also J2.3
- net VCC: now also R4.2, R9.2
- net EN_A: now reaches J1.2
- net EN_A: now also C9.2, R4.1
- net EN_B: now reaches J1.3
- net EN_B: now also C10.2, R9.1
Other:
- moved on the sheet: C7, J1, J2, R14

Commit message: udated by FZ
Connections:
- net VIB_CTRL: now reaches J2.9
- net VIB_CTRL: now also U1.D3 (P16)
Changed lines of the file:
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@@
+	(wire
+		(pts
+			(xy 223.52 96.52) (xy 231.14 96.52)
+		)
+		(stroke
+			(width 0)
+			(type default)
+		)
+	)
 	(wire
 		(pts
@@
 	(wire
 		(pts
-			(xy 100.33 54.61) (xy 110.49 54.61)
+			(xy 100.33 54.61) (xy 109.22 54.61)
 		)
 		(stroke
@@
 		(pts
 			(xy 186.69 39.37) (xy 186.69 41.91)
-		)
-		(stroke
-			(width 0)
-			(type default)
-		)
-	)
-	(wire
-		(pts
-			(xy 223.52 96.52) (xy 231.14 96.52)
 		)
 		(stroke
@@
 		)
 	)
+	(label "VIB_CTRL"
+		(at 109.22 54.61 180)
+		(fields_autoplaced yes)
+		(effects
+			(font
+				(size 1.27 1.27)
+			)
+			(justify right bottom)
+		)
+	)
 	(label "VBAT"
 		(at 74.93 158.75 0)
@@
 		(fields_autoplaced yes)
 		(effects
+			(font
+				(size 1.27 1.27)
+			)
+			(justify left bottom)
+		)
+	)
+	(label "VIB_CTRL"
+		(at 223.52 96.52 0)
+		(fields_autoplaced yes)
+		(effects
