File: PCB/CONN/V1/V1.kicad_pcb (KiCad board)
At the start: 2 copper layers, 28.9 x 23 mm, 3 parts, among them J1 Conn_01x06_Pin, J3 Conn_ARM_SWD_TagConnect_TC203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, U1 MCP73831-2-OT

Commit message: udated by FZ
Parts:
- added C1: 0.1uF, Capacitor_SMD:C_0402_1005Metric_Pad0.74x0.62mm_HandSolder, B.Cu at (105.4, 117.7)
- added C2: 10uF, Capacitor_SMD:C_0805_2012Metric_Pad1.18x1.45mm_HandSolder, B.Cu at (122.5, 116.7)
- added C3: 0.1uF, Capacitor_SMD:C_0402_1005Metric_Pad0.74x0.62mm_HandSolder, B.Cu at (107.9, 111.9)
- added C4: 10uF, Capacitor_SMD:C_0805_2012Metric_Pad1.18x1.45mm_HandSolder, B.Cu at (120.0, 113.6)
- added D1: LED_Small, LED_SMD:LED_0603_1608Metric_Pad1.05x0.95mm_HandSolder, F.Cu at (114.8, 107.5)
- added J2: Conn_01x10_Pin, Mylib:Pinheader_2mmx10, B.Cu at (114.5, 107.9)
- added J4: Conn_01x01_Pin, Mylib:1_pin, B.Cu at (117.8, 117.0)
- added J5: Conn_01x01_Pin, Mylib:1_pin, B.Cu at (105.1, 117.0)
- added J6: Conn_01x01_Pin, Mylib:1_pin, F.Cu at (116.3, 107.2)
- added J7: Conn_01x01_Pin, Mylib:1_pin, F.Cu at (110.0, 108.2)
- added J8: Conn_01x01_Pin, Mylib:1_pin, B.Cu at (122.3, 110.1)
- added J9: Conn_01x01_Pin, Mylib:1_pin, B.Cu at (126.2, 100.7)
- added Q1: DMN2056U, Package_TO_SOT_SMD:SOT-23, B.Cu at (123.1, 103.3)
- added R1: 470, Resistor_SMD:R_0402_1005Metric_Pad0.72x0.64mm_HandSolder, F.Cu at (114.8, 106.2)
- added R2: 10k, Resistor_SMD:R_0402_1005Metric_Pad0.72x0.64mm_HandSolder, B.Cu at (105.4, 115.8)
- added R3: 10k, Resistor_SMD:R_0402_1005Metric_Pad0.72x0.64mm_HandSolder, B.Cu at (122.0, 105.8)
- added SW1: CUS-12TB, Mylib:CUS-12B, B.Cu at (126.6, 117.0)
- U1: moved to B.Cu
- moved J3 1.37 mm to (114.5, 111.5)
- moved U1 1.30 mm to (108.6, 116.8), turned to 180 degrees
- moved J1 0.55 mm to (114.5, 103.0)
Connections:
- J1 pad 2: /BTN_3 -> /BTN_4
- J1 pad 3: /BTN_2 -> /BTN_3
- J1 pad 4: /BTN_1 -> /BTN_2
- J1 pad 5: /BTN_4 -> /BTN_1
- J3 pad 4: /SWCLK -> /SWDCLK
- U1 pad 3: Net-(J4-Pin_1) -> /VBAT
Routing:
- net VBUS: track 0.00 -> 28.9 mm, vias 0 -> 1
- net /VIN: track 0.00 -> 25.2 mm
- net Net-(U1-STAT): track 0.00 -> 21.3 mm, vias 0 -> 1
- net /VBAT: track 0.00 -> 15.7 mm
- net VCC: track 0.00 -> 14.8 mm, vias 0 -> 1
- net /BTN_4: track 0.00 -> 5.73 mm
- net /BTN_3: track 0.00 -> 5.73 mm
- net /BTN_2: track 0.00 -> 5.73 mm
- net /BTN_1: track 0.00 -> 5.73 mm
- net /SWDIO: track 0.00 -> 4.98 mm, vias 0 -> 1
- net /SWDCLK: track 0.00 -> 4.26 mm, vias 0 -> 1
- net /VIB_CTRL: track 0.00 -> 3.98 mm
- net Net-(J9-Pin_1): track 0.00 -> 2.21 mm
- net Net-(U1-PROG): track 0.00 -> 1.51 mm
- net Net-(D1-K): track 0.00 -> 1.43 mm
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- added copper zone on B.Cu, net GND
- added copper zone on F.Cu, net GND
Other:
- board text added: "+"
- board text added: "FZ. Liu"
- board text added: "MindCube"
